File: MODULO CNY70/MODULO CNY70.brd (EAGLE design)
At the start: 60.6 x 14 mm, 7 parts, among them T1 2N2222

Commit message: archivos actualizados
Routing:
- net N$4: track 80.9 -> 80.4 mm
- added copper zone on layer 16, net GND
- removed copper zone on layer 16, net 1
Other:
- board size 60.6 x 14 mm -> 54.3 x 16.5 mm
