File: PUENTE H/PUENTE H.brd (EAGLE design)
At the start: 83.5 x 62.2 mm, 20 parts, among them IC1 L293D, IC2 7805T

Commit message: archivos actualizados
Parts:
- moved LED1 124.1 mm to (-34.3, 53.3), turned to 0 degrees
- moved R1 115.9 mm to (-17.8, 64.8), turned to 0 degrees
- moved LED2 73.9 mm to (-47.0, 53.3), turned to 0 degrees
- moved R2 71.0 mm to (-27.9, 64.8), turned to 0 degrees
- moved MRIGT 12.5 mm to (72.4, 40.6)
- moved MLEFT 11.4 mm to (29.2, 40.6)
- moved D1 9.16 mm to (63.5, 44.5)
- moved D6 8.98 mm to (38.1, 44.5)
- moved D4 7.73 mm to (63.5, 39.4)
- moved D7 7.73 mm to (38.1, 39.4)
- moved D8 7.41 mm to (38.1, 36.8)
- moved D3 6.35 mm to (63.5, 36.8)
- moved ALIMENTACION 5.24 mm to (67.3, 19.1), turned to 180 degrees
- moved IC1 5.08 mm to (50.8, 40.6)
- moved D2 2.84 mm to (63.5, 41.9)
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Connections:
- net C1A: now also JP1.5; no longer JP1.2
- net C1B: now also JP1.4; no longer JP1.3
- net C2C: now also JP1.2; no longer JP1.4
- net C2D: now also JP1.3; no longer JP1.5
- net V12: no longer JP1.1
- net V5: now also JP1.1
Routing:
- net V12: track 356.6 -> 141.7 mm, vias 0 -> 6
- net V5: track 224.1 -> 123.6 mm, vias 0 -> 2
- net RIGT2: track 47.9 -> 18.6 mm
- net LEFT2: track 44.8 -> 18.6 mm
- net LEFT1: track 44.6 -> 18.6 mm
- net C2D: track 100.6 -> 75.3 mm
- net C1B: track 99.3 -> 74.3 mm
- net GND: track 282.7 -> 260.0 mm, vias 0 -> 2
- net RIGT1: track 39.2 -> 18.5 mm
- net C1A: track 13.8 -> 27.6 mm
- net C2C: track 13.7 -> 26.0 mm
- net N$5: track 5.08 -> 0.00 mm
- net N$2: track 5.08 -> 0.00 mm
- removed copper zone on layer 16, net 1
Other:
- board size 83.5 x 62.2 mm -> 63.2 x 67.3 mm
